File: Modules/I2C-OneWire_Probes/I2C-OneWire_Probes.brd (EAGLE design)
At the start: 69.8 x 18.4 mm, 25 parts, among them J1 QWIIC_RIGHT_ANGLE, Q1 AO3401, Q2 AO3401, Q3 AO3401, U1 AMS1117-3.3

Commit message: fixed pinout for 3.5mm jacks on I2C-OneWire-Probes
Parts:
- moved R7 0.63 mm to (15.9, 2.54)
Connections:
- net +3V3: now also U$2.P$4, U$3.P$4, U$4.P$4, U1.4; no longer U$2.P$1, U$3.P$1, U$4.P$1
- net GND: now also U$2.P$1, U$3.P$1, U$4.P$1; no longer U$2.P$5, U$3.P$5, U$4.P$5
- net N$3: now also U$2.P$5; no longer U$2.P$8
- net N$6: now also U$3.P$5; no longer U$3.P$8
- net N$9: now also U$4.P$5; no longer U$4.P$8
Routing:
- net +3V3: track 135.8 -> 126.6 mm
- net N$6: track 21.4 -> 12.9 mm
- net N$3: track 19.5 -> 12.0 mm, vias 2 -> 0
- net N$9: track 19.7 -> 12.6 mm
- net +5V: track 36.5 -> 42.9 mm
- net SDA: track 94.3 -> 91.0 mm, vias 3 -> 2
- net SCL: track 88.2 -> 86.0 mm, vias 4 -> 2
- net GND: track 29.0 -> 29.6 mm
Other:
- board text added: "I2C & OneWire Probe Board V0.2 Darkextratoasty Updated: 12/3/25"
- board text removed: "I2C & OneWire Probe Board V0.1 Darkextratoasty Updated: 1/16/25"
